File: electronic/rat_board.kicad_pcb (KiCad board)
At the start: 2 copper layers, 44.4 x 49.5 mm, 50 parts, among them P1 FRONT_LEFT_IR, P2 SIDE_LEFT_IR, P3 SIDE_RIGHT_IR, P4 FRONT_RIGHT_IR, P5 LEFT_MOTOR, P6 RIGHT_MOTOR, P7 JTAG, P8 IR_ARRAY, P9 CONN_02X03, SW1 SW_PUSH_SMALL_H, SW2 SWITCH_INV, SW3 SELECT_BUTTON, SW4 START_BUTTON, U1 TR05S3V3, U2 TB6612FNG, U3 STM32F103C8T6, Y1 32.768kHz, Y2 8MHz

Commit message: routing...
Parts:
- removed P8: IR_ARRAY, Pin_Headers:Pin_Header_Straight_1x11
- removed P9: CONN_02X03, Pin_Headers:Pin_Header_Straight_2x03
- added D6: LED_4, LEDs:LED-3MM, F.Cu at (68.7, 74.8)
- added D7: LED_5, LEDs:LED-3MM, F.Cu at (73.8, 74.8)
- added R11: 100, Resistors_SMD:R_0603_HandSoldering, F.Cu at (70.0, 71.6)
- added R12: 100, Resistors_SMD:R_0603_HandSoldering, F.Cu at (75.1, 71.6)
- added REF**: MountingHole_3.2mm_M3_Pad_Via, Mounting_Holes:MountingHole_3.2mm_M3_Pad_Via, F.Cu at (38.2, 32.9)
- added REF**: MountingHole_3.2mm_M3_Pad_Via, Mounting_Holes:MountingHole_3.2mm_M3_Pad_Via, F.Cu at (75.1, 32.9)
- D1: footprint LEDs:LED-5MM -> LEDs:LED-3MM
- D2: value POWER_LED -> LED_0; footprint LEDs:LED-5MM -> LEDs:LED-3MM
- D3: value POWER_LED -> LED_1; footprint LEDs:LED-5MM -> LEDs:LED-3MM
- D4: value POWER_LED -> LED_2; footprint LEDs:LED-5MM -> LEDs:LED-3MM
- D5: value POWER_LED -> LED_3; footprint LEDs:LED-5MM -> LEDs:LED-3MM
- moved 100nF2 176.5 mm to (44.7, 46.9)
- moved C7 164.0 mm to (38.4, 51.4), turned to 180 degrees
- moved R1 148.1 mm to (86.1, 33.8)
- moved 10nF1 138.0 mm to (29.6, 34.9)
- moved 0.1uF1 134.9 mm to (44.7, 43.6)
- moved 0.1uF2 124.1 mm to (37.6, 49.3), turned to 180 degrees
- moved 1uF1 123.6 mm to (29.6, 36.4)
- moved R9 122.3 mm to (44.7, 40.3)
- moved R2 121.2 mm to (38.2, 71.6)
- moved C_power2 120.8 mm to (37.6, 57.0)
- moved R6 119.9 mm to (37.6, 59.6)
- moved 4.7uF1 119.8 mm to (44.7, 45.2)
- moved C_power1 116.2 mm to (42.7, 57.0)
- moved R3 113.9 mm to (43.3, 71.6)
- moved R4 105.5 mm to (48.4, 71.6)
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Connections:
- net /USB_D+ renamed Net-(U3-Pad33)
- net /USB_D- renamed Net-(U3-Pad32)
- R10 pad 2: Net-(P9-Pad4) -> GND
- R9 pad 1: Net-(P9-Pad3) -> GND
- U2 pad 13: /VMN -> +BATT
- U2 pad 14: /VMN -> +BATT
- U2 pad 24: /VMN -> +BATT
- U3 pad 10: /ENC2A -> /ENC2B
- U3 pad 11: /ENC2B -> /ENC2A
- U3 pad 12: /IR5 -> Net-(U3-Pad12)
- U3 pad 13: /IR4 -> Net-(U3-Pad13)
- U3 pad 14: /IR3 -> Net-(U3-Pad14)
- U3 pad 15: /IR2 -> Net-(U3-Pad15)
- U3 pad 16: /IR1 -> /IR4
- U3 pad 17: /IR0 -> /IR3
- U3 pad 18: /M_PWMB -> /IR2
- U3 pad 19: /M_PWMA -> /IR1
- U3 pad 21: /M_AIN2 -> Net-(U3-Pad21)
- U3 pad 22: /M_AIN1 -> Net-(U3-Pad22)
- U3 pad 25: /M_STBY -> Net-(U3-Pad25)
- U3 pad 26: /M_BIN1 -> /LED0
- U3 pad 27: /M_BIN2 -> /LED1
- U3 pad 28: /LED0 -> /LED2
- U3 pad 29: /ENC1B -> /ENC1A
- U3 pad 30: /ENC1A -> /ENC1B
- U3 pad 31: /LED1 -> Net-(U3-Pad31)
- U3 pad 38: /LED2 -> /M_AIN2
- U3 pad 39: /LED3 -> /M_AIN1
- U3 pad 40: /BUZZER -> /M_STBY
- U3 pad 42: /TX1 -> /M_BIN1
- U3 pad 43: /RX1 -> /M_BIN2
- U3 pad 45: Net-(U3-Pad45) -> /M_PWMB
- U3 pad 46: /UB_START -> /M_PWMA
Routing:
- net /RESET: track 0.00 -> 49.1 mm, vias 0 -> 1
- net /LED0: track 0.00 -> 39.3 mm, vias 0 -> 2
- net /LED1: track 0.00 -> 38.3 mm, vias 0 -> 2
- net /LED2: track 0.00 -> 32.8 mm
- net /IR3: track 35.3 -> 6.18 mm
- net +BATT: track 0.00 -> 26.6 mm, vias 0 -> 1
- net /UB_SELECT: track 0.00 -> 26.2 mm, vias 0 -> 1
- net /IR2: track 32.3 -> 7.82 mm
- net /IR4: track 36.2 -> 12.5 mm
- net /SWDIO: track 0.00 -> 23.6 mm, vias 0 -> 1
- net /ENC2A: track 0.00 -> 23.0 mm, vias 0 -> 1
- net /ENC1A: track 0.00 -> 20.2 mm
- net /SWDCLK: track 0.00 -> 20.0 mm, vias 0 -> 1
- net /ENC2B: track 0.00 -> 19.6 mm, vias 0 -> 1
- net /BOOT0: track 0.00 -> 17.1 mm, vias 0 -> 2
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Other:
- board size 44.4 x 49.5 mm -> 44.5 x 49.5 mm
- net class lipo added: clearance 0.2, trace_width 0.8, via_dia 0.6, via_drill 0.4
- net class motors added: clearance 0.2, trace_width 0.4, via_dia 0.6, via_drill 0.4

Commit message: updated pcb
Parts:
- removed D1: POWER_LED, LEDs:LED-3MM
- removed R1: 100, Resistors_SMD:R_0603_HandSoldering
- SW2: footprint Buttons_Switches_ThroughHole:SW_Micro_SPST -> Connect:Wafer_Vertical10x5.8x7RM2.5-3
- U1: footprint Pin_Headers:Pin_Header_Angled_1x03 -> Connect:Wafer_Vertical10x5.8x7RM2.5-3
- Y1: footprint Crystals:Crystal_MC-156 -> Crystals:Crystal_MC-306
- moved 10nF1 21.3 mm to (49.0, 43.7), turned to 90 degrees
- moved 1uF1 19.6 mm to (47.8, 43.7), turned to 90 degrees
- moved C7 19.1 mm to (48.3, 67.8), turned to 0 degrees
- moved C2 17.4 mm to (65.3, 67.8), turned to 0 degrees
- moved C_power2 16.0 mm to (46.5, 43.7), turned to 90 degrees
- moved R6 16.0 mm to (46.5, 46.2), turned to 180 degrees
- moved C_power1 13.6 mm to (45.2, 43.7), turned to 90 degrees
- moved C1 12.7 mm to (46.5, 47.5)
- moved 0.1uF2 8.90 mm to (46.5, 48.8), turned to 0 degrees
- moved 100nF2 6.75 mm to (45.2, 40.1), turned to 270 degrees
- moved R9 5.59 mm to (50.3, 40.1), turned to 90 degrees
- moved 4.7uF1 5.38 mm to (46.5, 40.1), turned to 270 degrees
- moved 100nF1 4.67 mm to (49.0, 40.1), turned to 270 degrees
- moved 0.1uF1 4.59 mm to (47.8, 40.1), turned to 270 degrees
- moved Y1 3.95 mm to (71.1, 44.5), turned to 90 degrees
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Connections:
- P1 pad 3: /3V3 -> +3V3
- P2 pad 3: /3V3 -> +3V3
- P3 pad 3: /3V3 -> +3V3
- P4 pad 3: /3V3 -> +3V3
- P5 pad 2: /3V3 -> +3V3
- P6 pad 2: /3V3 -> +3V3
- SW2 pad 1: +BATT -> Net-(SW2-Pad1)
- SW2 pad 3: /VUSB -> +BATT
- U2 pad 20: /3V3 -> +3V3
- U3 pad 1: /3V3 -> +3V3
- U3 pad 10: /ENC2B -> /ENC2A
- U3 pad 11: /ENC2A -> /ENC2B
- U3 pad 13: Net-(U3-Pad13) -> /LED3
- U3 pad 14: Net-(U3-Pad14) -> /LED4
- U3 pad 15: Net-(U3-Pad15) -> /LED5
- U3 pad 2: Net-(U3-Pad2) -> /UB_START
- U3 pad 24: /3V3 -> +3V3
- U3 pad 36: /3V3 -> +3V3
- U3 pad 48: /3V3 -> +3V3
- U3 pad 9: /3V3 -> +3V3
Routing:
- net /LED5: track 0.00 -> 56.3 mm
- net /LED3: track 0.00 -> 53.1 mm, vias 0 -> 2
- net /LED4: track 0.00 -> 50.8 mm, vias 0 -> 2
- net /RESET: track 49.1 -> 6.98 mm, vias 1 -> 0
- net /LED0: track 39.3 -> 0.04 mm, vias 2 -> 0
- net /LED1: track 38.3 -> 0.59 mm, vias 2 -> 0
- net /UB_START: track 10.0 -> 47.2 mm
- net +BATT: track 26.6 -> 57.6 mm, vias 1 -> 2
- net +3V3: track 0.00 -> 26.5 mm, vias 0 -> 6
- net /M_PWMA: track 0.00 -> 16.3 mm, vias 0 -> 2
- net /BOOT1: track 13.1 -> 0.00 mm
- net Net-(C5-Pad2): track 0.00 -> 11.5 mm
- net /UB_SELECT: track 26.2 -> 32.7 mm
- net Net-(C3-Pad2): track 0.00 -> 6.11 mm
- net /ENC2A: track 23.0 -> 19.1 mm
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- added copper zone on B.Cu, net +3V3
- added copper zone on F.Cu, net GND
Other:
- net class lipo: trace_width 0.8 -> 1
- net class motors: trace_width 0.4 -> 1

Commit message: updated pcb
Parts:
- removed 0.1uF1, 0.1uF2, 100nF1, 100nF2, 10nF1, 1uF1, 4.7uF1, C1, C_power1, C_power2: C, Capacitors_SMD:C_0603_HandSoldering
- removed C2, C7: 10uF, SMD_Packages:SMD-1206_Pol
- removed C3, C4, C5, C6: 20p, Capacitors_SMD:C_0603_HandSoldering
- removed U1: TR05S3V3, Connect:Wafer_Vertical10x5.8x7RM2.5-3
- removed ext1: R, Resistors_SMD:R_0603_HandSoldering
- added ?: 20p, Capacitors_SMD:C_0603_HandSoldering, F.Cu at (65.9, 43.2)
- added ?: 20p, Capacitors_SMD:C_0603_HandSoldering, F.Cu at (65.9, 47.0)
- added ?: 20p, Capacitors_SMD:C_0603_HandSoldering, F.Cu at (65.9, 45.7)
- added ?: 10uF, SMD_Packages:SMD-1206_Pol, F.Cu at (65.0, 67.6)
- added ?: C, Capacitors_SMD:C_0603_HandSoldering, F.Cu at (45.7, 48.0)
- added ?: 100nF, Capacitors_SMD:C_0603_HandSoldering, F.Cu at (45.7, 45.2)
- added ?: 100nF, Capacitors_SMD:C_0603_HandSoldering, F.Cu at (45.7, 43.9)
- added ?: 4.7uF, Capacitors_SMD:C_0603_HandSoldering, F.Cu at (65.9, 48.3)
- added ?: 10nF, Capacitors_SMD:C_0603_HandSoldering, F.Cu at (49.8, 39.9)
- added ?: 1uF, Capacitors_SMD:C_0603_HandSoldering, F.Cu at (48.5, 39.9)
- added ?: 20p, Capacitors_SMD:C_0603_HandSoldering, F.Cu at (65.9, 44.5)
- added ?: R, Resistors_SMD:R_0603_HandSoldering, F.Cu at (65.8, 41.8)
- added ?: 0.1uF, Capacitors_SMD:C_0805, F.Cu at (47.2, 69.6)
- added ?: 0.1uF, Capacitors_SMD:C_0805, F.Cu at (66.0, 69.6)
- added ?: TR05S3V3, custom-lib:TR05S3V3, F.Cu at (38.1, 41.9)
- added C14: 10uF, SMD_Packages:SMD-1206_Pol, F.Cu at (48.3, 67.6)
- added DC-DC: CONN_01X02, Socket_Strips:Socket_Strip_Straight_1x02, F.Cu at (45.7, 41.9)
- moved R9 2.62 mm to (52.6, 38.9), turned to 0 degrees
- moved ? 1.09 mm to (70.7, 45.5)
- moved ? 0.92 mm to (45.7, 46.7)
- moved ? 0.80 mm to (65.8, 40.4)
- moved ? 0.52 mm to (40.1, 32.9)
- moved ? 0.40 mm to (75.9, 42.9)
- moved ? 0.28 mm to (73.2, 32.9)
- renumbered P7 to ?, R3 to ?, R4 to ?, R5 to ?, R7 to ?, R8 to ?, R10 to ?, Y2 to ?, R11 to ?, R12 to ?, REF** to ?, U2 to ?, U3 to ?, Y1 to ?, R6 to ?, R2 to ?, D2 to L1, D3 to L2, D4 to L3, D5 to L4, D6 to L5, D7 to L6, P5 to MOTOR, P6 to MOTOR, P1 to S1, P2 to S2, P3 to S3, P4 to S4
Routing:
- net /RESET: track 6.98 -> 52.9 mm, vias 0 -> 2
- net /LED0: track 0.04 -> 37.7 mm
- net /LED1: track 0.59 -> 33.8 mm
- net +BATT: track 57.6 -> 74.7 mm, vias 2 -> 3
- net +3V3: track 26.5 -> 41.3 mm, vias 6 -> 8
- net Net-(SW2-Pad2): track 0.00 -> 11.9 mm
- net /UB_START: track 47.2 -> 39.1 mm
- net GND: track 0.00 -> 8.00 mm
- net /LED5: track 56.3 -> 50.3 mm, vias 0 -> 2
- net /BOOT1: track 0.00 -> 3.84 mm
- net Net-(C6-Pad1): track 2.68 -> 0.00 mm
- net Net-(C8-Pad1): track 0.00 -> 2.50 mm
- net /OSC32IN: track 5.09 -> 4.12 mm
- net /OSCOUT: track 7.51 -> 6.57 mm
- net /LED3: track 53.1 -> 52.4 mm
Other:
- board size 44.5 x 49.5 mm -> 43.2 x 48.3 mm
