File: electronic/rat_board.sch (KiCad schematic (older format))
At the start: 57 parts

Commit message: updates in pcb
Parts:
- removed D? (x2): POWER_LED, symbol LED
- removed P?: USB, symbol USB_OTG
- removed R? (x4): 100, symbol R
- removed R?: 1.5k, symbol R
- added P8: IR_ARRAY, Pin_Headers:Pin_Header_Straight_1x11, symbol CONN_01X11
- 0.1uF1: renamed from 0.1uF?; footprint (none) -> Capacitors_SMD:C_0603_HandSoldering
- 0.1uF2: renamed from 0.1uF; footprint (none) -> Capacitors_SMD:C_0603_HandSoldering
- 100nF1, 100nF2: renamed from 100nF; footprint (none) -> Capacitors_SMD:C_0603_HandSoldering
- 10nF1: renamed from 10nF; footprint (none) -> Capacitors_SMD:C_0603_HandSoldering
- 1uF1: renamed from 1uF; footprint (none) -> Capacitors_SMD:C_0603_HandSoldering
- 4.7uF1: renamed from 4.7uF; footprint (none) -> Capacitors_SMD:C_0603_HandSoldering
- C1, C3, C4, C5, C6: renamed from C?; footprint (none) -> Capacitors_SMD:C_0603_HandSoldering
- C2, C7: renamed from C?; footprint (none) -> SMD_Packages:SMD-1206_Pol
- C_power1, C_power2: renamed from C_power; footprint (none) -> Capacitors_SMD:C_0603_HandSoldering
- D1, D2, D3, D4, D5: renamed from D?; footprint (none) -> LEDs:LED-5MM
- P1, P2, P3, P4: renamed from P?; footprint (none) -> Pin_Headers:Pin_Header_Straight_1x03
- P5, P6: renamed from P?; footprint (none) -> Pin_Headers:Pin_Header_Straight_1x06
- P7: renamed from P?; footprint (none) -> Pin_Headers:Pin_Header_Angled_1x04
- P9: renamed from P?; footprint (none) -> Pin_Headers:Pin_Header_Straight_2x03
- R1, R10, R2, R3, R4, R5, R6, R7, R8, R9: renamed from R?; footprint (none) -> Resistors_SMD:R_0603_HandSoldering
- SW1, SW3, SW4: renamed from SW?; footprint (none) -> Buttons_Switches_ThroughHole:SW_PUSH_6mm
- SW2: renamed from SW?; footprint (none) -> Buttons_Switches_ThroughHole:SW_Micro_SPST
- U1: renamed from U?; footprint (none) -> Pin_Headers:Pin_Header_Angled_1x03
- U2: renamed from U?; footprint (none) -> Housings_SSOP:SSOP-24_5.3x8.2mm_Pitch0.65mm
- U3: renamed from U?; footprint LQFP48_7X7MM_0.5MMPP -> Housings_QFP:LQFP-48_7x7mm_Pitch0.5mm
- Y1: renamed from Y?; footprint (none) -> Crystals:Crystal_MC-156
- Y2: renamed from Y?; footprint (none) -> Crystals:Crystal_HC50-U_Vertical
- ext1: renamed from ext; footprint (none) -> Resistors_SMD:R_0603_HandSoldering
Connections:
- net labels added: BUZZER, INPUT_A, INPUT_B, IR0, IR5, LED0, M_A01, M_A02, M_AIN1, M_AIN2, M_B01, M_B02, M_BIN1, M_BIN2, M_PWMA, M_PWMB, M_STBY, RX1, TX1, VMN
- net labels removed: 5V, A01, A02, AIN1_d, AIN2_d, B01, B02, BIN1, BIN2, LED4, LED5, LED6, M1A, M1B, M2A, M2B, PWM_M1, PWM_M2, STBY, VDD1
- wire segments 180 -> 201
- no-connect marks 2 -> 0
Other:
- note added: "IR_ARRAY"
- note removed: "USB CONNECTOR"
- moved on the sheet: C_power1, C_power2, SW2, U1

Commit message: routing...
Parts:
- removed P8: IR_ARRAY, Pin_Headers:Pin_Header_Straight_1x11, symbol CONN_01X11
- removed P9: CONN_02X03, Pin_Headers:Pin_Header_Straight_2x03, symbol CONN_02X03
- added D6: LED_4, LEDs:LED-3MM, symbol LED
- added D7: LED_5, LEDs:LED-3MM, symbol LED
- added R11, R12: 100, Resistors_SMD:R_0603_HandSoldering, symbol R
- D1: footprint LEDs:LED-5MM -> LEDs:LED-3MM
- D2: value POWER_LED -> LED_0; footprint LEDs:LED-5MM -> LEDs:LED-3MM
- D3: value POWER_LED -> LED_1; footprint LEDs:LED-5MM -> LEDs:LED-3MM
- D4: value POWER_LED -> LED_2; footprint LEDs:LED-5MM -> LEDs:LED-3MM
- D5: value POWER_LED -> LED_3; footprint LEDs:LED-5MM -> LEDs:LED-3MM
Connections:
- net labels added: LED4, LED5
- net labels removed: BUZZER, INPUT_A, INPUT_B, IR0, IR5, RX1, TX1, USB_D+, USB_D-, VMN
- wire segments 201 -> 190
Other:
- note removed: "IR_ARRAY"

Commit message: updated pcb
Parts:
- removed D1: POWER_LED, LEDs:LED-3MM, symbol LED
- removed R1: 100, Resistors_SMD:R_0603_HandSoldering, symbol R
- added P8: CONN_01X02, Socket_Strips:Socket_Strip_Straight_1x02, symbol CONN_01X02
- SW2: footprint Buttons_Switches_ThroughHole:SW_Micro_SPST -> Connect:Wafer_Vertical10x5.8x7RM2.5-3
Connections:
- net labels removed: VUSB
- wire segments 190 -> 187
- no-connect marks 0 -> 1

Commit message: updated pcb
Parts:
- removed C_power1, C_power2: C, Capacitors_SMD:C_0603_HandSoldering, symbol C
- C11: renamed from 0.1uF1; value C -> 0.1uF
- C13: renamed from 0.1uF2; value C -> 0.1uF
- C2: renamed from 100nF1; value C -> 100nF
- C3: renamed from 100nF2; value C -> 100nF
- C4: renamed from 4.7uF1; value C -> 4.7uF
- C5: renamed from 10nF1; value C -> 10nF
- C6: renamed from 1uF1; value C -> 1uF
- SW2: footprint Connect:Wafer_Vertical10x5.8x7RM2.5-3 -> custom-lib:TR05S3V3
- renumbered C4 to C10, C2 to C12, C7 to C14, C5 to C7, C6 to C8, C3 to C9
Connections:
- wire segments 187 -> 186
- no-connect marks 1 -> 8
Changed lines of the file:
@@
 OSC32OUT
 $Comp
-L C 0.1uF2
+L C C13
 U 1 1 5878F688
 P 10300 5900
-F 0 "0.1uF2" H 10325 6000 50  0000 L CNN
-F 1 "C" H 10325 5800 50  0000 L CNN
+F 0 "C13" H 10325 6000 50  0000 L CNN
+F 1 "0.1uF" H 10325 5800 50  0000 L CNN
 F 2 "Capacitors_SMD:C_0603_HandSoldering" H 10338 5750 50  0001 C CNN
 F 3 "" H 10300 5900 50  0000 C CNN
@@
 $EndComp
 $Comp
-L C 100nF1
+L C C2
 U 1 1 5878F74F
 P 9500 1650
-F 0 "100nF1" H 9525 1750 50  0000 L CNN
-F 1 "C" H 9525 1550 50  0000 L CNN
+F 0 "C2" H 9525 1750 50  0000 L CNN
+F 1 "100nF" H 9525 1550 50  0000 L CNN
 F 2 "Capacitors_SMD:C_0603_HandSoldering" H 9538 1500 50  0001 C CNN
 F 3 "" H 9500 1650 50  0000 C CNN
@@
 $EndComp
 $Comp
-L C 100nF2
+L C C3
 U 1 1 5878F78C
 P 9800 1650
-F 0 "100nF2" H 9825 1750 50  0000 L CNN
-F 1 "C" H 9825 1550 50  0000 L CNN
+F 0 "C3" H 9825 1750 50  0000 L CNN
+F 1 "100nF" H 9825 1550 50  0000 L CNN
 F 2 "Capacitors_SMD:C_0603_HandSoldering" H 9838 1500 50  0001 C CNN
 F 3 "" H 9800 1650 50  0000 C CNN
@@
 $EndComp
 $Comp
-L C 10nF1
+L C C5
 U 1 1 5878F7CC
 P 10400 1650
-F 0 "10nF1" H 10425 1750 50  0000 L CNN
-F 1 "C" H 10425 1550 50  0000 L CNN
+F 0 "C5" H 10425 1750 50  0000 L CNN
+F 1 "10nF" H 10425 1550 50  0000 L CNN
 F 2 "Capacitors_SMD:C_0603_HandSoldering" H 10438 1500 50  0001 C CNN
 F 3 "" H 10400 1650 50  0000 C CNN
@@
 $EndComp
 $Comp
-L C C5
+L C C7
 U 1 1 5878FF91
 P 10400 2850
-F 0 "C5" H 10425 2950 50  0000 L CNN
+F 0 "C7" H 10425 2950 50  0000 L CNN
 F 1 "20p" H 10425 2750 50  0000 L CNN
 F 2 "Capacitors_SMD:C_0603_HandSoldering" H 10438 2700 50  0001 C CNN
@@
 $EndComp
 $Comp
-L C C6
+L C C8
 U 1 1 5879018F
 P 10400 3350
-F 0 "C6" H 10425 3450 50  0000 L CNN
+F 0 "C8" H 10425 3450 50  0000 L CNN
 F 1 "20p" H 10425 3250 50  0000 L CNN
 F 2 "Capacitors_SMD:C_0603_HandSoldering" H 10438 3200 50  0001 C CNN
@@
 OSCOUT
 $Comp
-L C C3
+L C C9
 U 1 1 58790916
 P 10100 3850
-F 0 "C3" H 10125 3950 50  0000 L CNN
+F 0 "C9" H 10125 3950 50  0000 L CNN
 F 1 "20p" H 10125 3750 50  0000 L CNN
 F 2 "Capacitors_SMD:C_0603_HandSoldering" H 10138 3700 50  0001 C CNN
@@
 $EndComp
 $Comp
-L C C4
+L C C10
 U 1 1 58790922
 P 10100 4350
-F 0 "C4" H 10125 4450 50  0000 L CNN
+F 0 "C10" H 10125 4450 50  0000 L CNN
 F 1 "20p" H 10125 4250 50  0000 L CNN
 F 2 "Capacitors_SMD:C_0603_HandSoldering" H 10138 4200 50  0001 C CNN
@@
 $EndComp
 $Comp
-L C 4.7uF1
+L C C4
 U 1 1 587915B6
 P 10100 1650
-F 0 "4.7uF1" H 10125 1750 50  0000 L CNN
-F 1 "C" H 10125 1550 50  0000 L CNN
+F 0 "C4" H 10125 1750 50  0000 L CNN
+F 1 "4.7uF" H 10125 1550 50  0000 L CNN
 F 2 "Capacitors_SMD:C_0603_HandSoldering" H 10138 1500 50  0001 C CNN
 F 3 "" H 10100 1650 50  0000 C CNN
@@
 	1    0    0    -1
 $EndComp
-Text Label 10300 5650 1    60   ~ 0
-VMX
 Text Label 9500 1400 1    60   ~ 0
 VDD2
@@
 GND
 $Comp
-L C 1uF1
+L C C6
 U 1 1 58792524
 P 10700 1650
-F 0 "1uF1" H 10725 1750 50  0000 L CNN
-F 1 "C" H 10725 1550 50  0000 L CNN
+F 0 "C6" H 10725 1750 50  0000 L CNN
+F 1 "1uF" H 10725 1550 50  0000 L CNN
 F 2 "Capacitors_SMD:C_0603_HandSoldering" H 10738 1500 50  0001 C CNN
 F 3 "" H 10700 1650 50  0000 C CNN
@@
 	1    0    0    -1
 $EndComp
-Text Label 10600 5650 1    60   ~ 0
+Text Label 10600 5600 1    60   ~ 0
 VMX
 $Comp
-L CP1 C7
+L CP1 C14
 U 1 1 58799BC8
 P 10600 5900
-F 0 "C7" H 10625 6000 50  0000 L CNN
+F 0 "C14" H 10625 6000 50  0000 L CNN
 F 1 "10uF" H 10625 5800 50  0000 L CNN
 F 2 "SMD_Packages:SMD-1206_Pol" H 10600 5900 50  0001 C CNN
@@
 $Comp
 L +BATT #PWR022
-U 1 1 58799EB8
-P 10300 5300
-F 0 "#PWR022" H 10300 5150 50  0001 C CNN
-F 1 "+BATT" H 10300 5440 50  0000 C CNN
-F 2 "" H 10300 5300 50  0000 C CNN
-F 3 "" H 10300 5300 50  0000 C CNN
-	1    10300 5300
-	1    0    0    -1
-$EndComp
-$Comp
-L +BATT #PWR023
 U 1 1 58799F36
 P 10600 5300
-F 0 "#PWR023" H 10600 5150 50  0001 C CNN
+F 0 "#PWR022" H 10600 5150 50  0001 C CNN
 F 1 "+BATT" H 10600 5440 50  0000 C CNN
 F 2 "" H 10600 5300 50  0000 C CNN
@@
 $EndComp
 $Comp
-L C 0.1uF1
+L C C11
 U 1 1 5879A0ED
 P 9650 5900
-F 0 "0.1uF1" H 9675 6000 50  0000 L CNN
-F 1 "C" H 9675 5800 50  0000 L CNN
+F 0 "C11" H 9675 6000 50  0000 L CNN
+F 1 "0.1uF" H 9675 5800 50  0000 L CNN
 F 2 "Capacitors_SMD:C_0603_HandSoldering" H 9688 5750 50  0001 C CNN
 F 3 "" H 9650 5900 50  0000 C CNN
@@
 $EndComp
 $Comp
-L GND #PWR024
+L GND #PWR023
 U 1 1 5879A0F3
 P 9650 6050
-F 0 "#PWR024" H 9650 5800 50  0001 C CNN
+F 0 "#PWR023" H 9650 5800 50  0001 C CNN
 F 1 "GND" H 9650 5900 50  0000 C CNN
 F 2 "" H 9650 6050 50  0000 C CNN
@@
 $EndComp
 $Comp
-L GND #PWR025
+L GND #PWR024
 U 1 1 5879A0FB
 P 9950 6050
-F 0 "#PWR025" H 9950 5800 50  0001 C CNN
+F 0 "#PWR024" H 9950 5800 50  0001 C CNN
 F 1 "GND" H 9950 5900 50  0000 C CNN
 F 2 "" H 9950 6050 50  0000 C CNN
@@
 $EndComp
 $Comp
-L CP1 C2
+L CP1 C12
 U 1 1 5879A103
 P 9950 5900
-F 0 "C2" H 9975 6000 50  0000 L CNN
+F 0 "C12" H 9975 6000 50  0000 L CNN
 F 1 "10uF" H 9975 5800 50  0000 L CNN
 F 2 "SMD_Packages:SMD-1206_Pol" H 9950 5900 50  0001 C CNN
@@
 Text Label 8450 5350 2    60   ~ 0
 3V3
-Text Label 9650 5650 1    60   ~ 0
-VCC_d
-Text Label 9950 5650 1    60   ~ 0
+Text Label 9950 5600 1    60   ~ 0
 VCC_d
 $Comp
@@
 $EndComp
 $Comp
-L +3V3 #PWR026
+L +3V3 #PWR025
 U 1 1 5879F86D
 P 3900 1650
-F 0 "#PWR026" H 3900 1500 50  0001 C CNN
+F 0 "#PWR025" H 3900 1500 50  0001 C CNN
 F 1 "+3V3" H 3900 1790 50  0000 C CNN
 F 2 "" H 3900 1650 50  0000 C CNN
@@
 $EndComp
 $Comp
-L GND #PWR027
+L GND #PWR026
 U 1 1 587A02F5
 P 5050 1800
-F 0 "#PWR027" H 5050 1550 50  0001 C CNN
+F 0 "#PWR026" H 5050 1550 50  0001 C CNN
 F 1 "GND" H 5050 1650 50  0000 C CNN
 F 2 "" H 5050 1800 50  0000 C CNN
@@
 $EndComp
 $Comp
-L +3V3 #PWR028
+L +3V3 #PWR027
 U 1 1 587A0699
 P 3900 1050
-F 0 "#PWR028" H 3900 900 50  0001 C CNN
+F 0 "#PWR027" H 3900 900 50  0001 C CNN
 F 1 "+3V3" H 3900 1190 50  0000 C CNN
 F 2 "" H 3900 1050 50  0000 C CNN
@@
 $EndComp
 $Comp
-L GND #PWR029
+L GND #PWR028
 U 1 1 587A069F
 P 5050 1200
-F 0 "#PWR029" H 5050 950 50  0001 C CNN
+F 0 "#PWR028" H 5050 950 50  0001 C CNN
 F 1 "GND" H 5050 1050 50  0000 C CNN
 F 2 "" H 5050 1200 50  0000 C CNN
@@
 USER BUTTONS
 $Comp
-L +3V3 #PWR030
-U 1 1 587A0486
-P 9650 5300
-F 0 "#PWR030" H 9650 5150 50  0001 C CNN
-F 1 "+3V3" H 9650 5440 50  0000 C CNN
-F 2 "" H 9650 5300 50  0000 C CNN
-F 3 "" H 9650 5300 50  0000 C CNN
-	1    9650 5300
-	1    0    0    -1
-$EndComp
-$Comp
-L +3V3 #PWR031
+L +3V3 #PWR029
 U 1 1 587A06CD
 P 9950 5300
-F 0 "#PWR031" H 9950 5150 50  0001 C CNN
+F 0 "#PWR029" H 9950 5150 50  0001 C CNN
 F 1 "+3V3" H 9950 5440 50  0000 C CNN
 F 2 "" H 9950 5300 50  0000 C CNN
@@
 $EndComp
 $Comp
-L +3V3 #PWR032
+L +3V3 #PWR030
 U 1 1 587A133C
 P 4550 5600
-F 0 "#PWR032" H 4550 5450 50  0001 C CNN
+F 0 "#PWR030" H 4550 5450 50  0001 C CNN
 F 1 "+3V3" H 4550 5740 50  0000 C CNN
 F 2 "" H 4550 5600 50  0000 C CNN
@@
 $EndComp
 $Comp
-L C C_power2
-U 1 1 587A19DE
-P 4550 5850
-F 0 "C_power2" H 4575 5950 50  0000 L CNN
-F 1 "C" H 4575 5750 50  0000 L CNN
-F 2 "Capacitors_SMD:C_0603_HandSoldering" H 4588 5700 50  0001 C CNN
-F 3 "" H 4550 5850 50  0000 C CNN
-	1    4550 5850
-	1    0    0    -1
-$EndComp
-$Comp
-L C C_power1
-U 1 1 587A1A99
-P 3250 5850
-F 0 "C_power1" H 3275 5950 50  0000 L CNN
-F 1 "C" H 3275 5750 50  0000 L CNN
-F 2 "Capacitors_SMD:C_0603_HandSoldering" H 3288 5700 50  0001 C CNN
-F 3 "" H 3250 5850 50  0000 C CNN
-	1    3250 5850
-	1    0    0    -1
-$EndComp
-$Comp
-L GND #PWR033
+L GND #PWR031
 U 1 1 587A1C89
 P 3900 6100
-F 0 "#PWR033" H 3900 5850 50  0001 C CNN
+F 0 "#PWR031" H 3900 5850 50  0001 C CNN
 F 1 "GND" H 3900 5950 50  0000 C CNN
 F 2 "" H 3900 6100 50  0000 C CNN
@@
 $EndComp
 $Comp
-L +BATT #PWR034
+L +BATT #PWR032
 U 1 1 587A66DA
 P 4350 4650
-F 0 "#PWR034" H 4350 4500 50  0001 C CNN
+F 0 "#PWR032" H 4350 4500 50  0001 C CNN
 F 1 "+BATT" H 4350 4790 50  0000 C CNN
 F 2 "" H 4350 4650 50  0000 C CNN
@@
 Wire Wire Line
 	10750 2850 10750 2950
-Wire Wire Line
-	10300 5300 10300 5750
 Wire Wire Line
 	9500 1500 9500 1050
@@
 Wire Wire Line
 	10600 5300 10600 5750
-Wire Wire Line
-	9650 5300 9650 5750
 Wire Wire Line
 	9950 5300 9950 5750
@@
 	4550 5700 4550 5600
 Wire Wire Line
-	3250 6000 3250 6050
-Wire Wire Line
-	3250 6050 4550 6050
-Wire Wire Line
-	4550 6050 4550 6000
-Wire Wire Line
 	3900 6000 3900 6100
-Connection ~ 3900 6050
 Wire Wire Line
 	8350 2600 8750 2600
@@
 Text Label 6850 4100 1    60   ~ 0
 LED5
-Text Label 4300 6050 2    60   ~ 0
-GND
 Wire Wire Line
 	4350 4650 4350 5100
@@
 Connection ~ 4350 4800
 $Comp
-L GND #PWR035
+L GND #PWR033
 U 1 1 588D1781
 P 4600 5100
-F 0 "#PWR035" H 4600 4850 50  0001 C CNN
+F 0 "#PWR033" H 4600 4850 50  0001 C CNN
 F 1 "GND" H 4600 4950 50  0000 C CNN
 F 2 "" H 4600 5100 50  0000 C CNN
@@
 F 0 "SW2" H 3550 5150 50  0000 C CNN
 F 1 "SWITCH_INV" H 3600 4850 50  0000 C CNN
-F 2 "Connect:Wafer_Vertical10x5.8x7RM2.5-3" H 3750 5000 50  0001 C CNN
+F 2 "custom-lib:TR05S3V3" H 3750 5000 50  0001 C CNN
 F 3 "" H 3750 5000 50  0000 C CNN
 	1    3750 5000
@@
 	4350 5100 4250 5100
 NoConn ~ 4250 4900
+Text Label 3900 6100 0    60   ~ 0
+GND
+Wire Wire Line
+	9650 5750 9650 5650
+Wire Wire Line
+	9650 5650 9950 5650
+Connection ~ 9950 5650
+Wire Wire Line
+	10300 5750 10300 5650
+Wire Wire Line
+	10300 5650 10600 5650
+Connection ~ 10600 5650
+NoConn ~ 8750 2300
+NoConn ~ 8750 2400
+NoConn ~ 8750 2500
+NoConn ~ 8750 3100
+NoConn ~ 5650 3100
+NoConn ~ 7450 4100
+NoConn ~ 7550 4100
 $EndSCHEMATC
